File: Controller/Controller.kicad_sch (KiCad schematic)
At the start: 63 parts, among them J1 UART, J2 NTC Conn, J3 PWR, J4 Heater, J5 PM1, J6 Pololu reg17a 5V, J7 PM2, Q1 BC547, Q2 BC547, Q3 IRF5305, SW5 Reset, U3 LM324, U4 LM393, U6 ProMicro

Commit message: Suppress backfeeding from Vbus to +5V rail
Parts:
- added D4: 1N5817, Diode_THT:D_DO-41_SOD81_P10.16mm_Horizontal, symbol Diode:1N5817
Connections:
- net +5V: now also D4.2 (A); no longer C22.1, J7.4 (Pin_4), U6.21 (VCC)
- new net: C22.1, D4.1 (K), J7.4 (Pin_4), U6.21 (VCC)
Other:
- note added: "Suppress backfeeding from VBus to +5V rail"
Changed lines of the file:
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@@
 		)
 	)
+	(text "Suppress backfeeding\nfrom VBus to +5V rail"
+		(exclude_from_sim no)
+		(at 124.46 138.43 0)
+		(effects
+			(font
+				(size 1.27 1.27)
+			)
+		)
+	)
 	(text "STAR GND at shunt/PSU return region.\nKeep heater current out of analog and MCU ground paths.\nRun separate returns for:\n- heater/shunt\n- analog circuitry\n- Pro Micro / digital\n- 5 V buck"
 		(exclude_from_sim yes)
@@
 	(wire
 		(pts
-			(xy 111.76 138.43) (xy 111.76 140.97)
-		)
-		(stroke
-			(width 0)
-			(type default)
-		)
-	)
-	(wire
-		(pts
 			(xy 97.79 92.71) (xy 97.79 110.49)
 		)
@@
 	(wire
 		(pts
+			(xy 100.33 140.97) (xy 104.14 140.97)
+		)
+		(stroke
+			(width 0)
+			(type default)
+		)
+	)
+	(wire
+		(pts
 			(xy 40.64 62.23) (xy 40.64 63.5)
 		)
@@
 	(wire
 		(pts
+			(xy 100.33 138.43) (xy 100.33 140.97)
+		)
+		(stroke
+			(width 0)
+			(type default)
+		)
+	)
+	(wire
+		(pts
 			(xy 135.89 77.47) (xy 146.05 77.47)
 		)
@@
 	(symbol
 		(lib_id "power:+5V")
-		(at 111.76 138.43 0)
+		(at 100.33 138.43 0)
 		(unit 1)
 		(body_style 1)
@@
 		(fields_autoplaced yes)
 		(property "Reference" "#PWR071"
-			(at 111.76 142.24 0)
+			(at 100.33 142.24 0)
 			(hide yes)
 			(show_name no)
@@
 		)
 		(property "Value" "+5V"
-			(at 111.76 134.2969 0)
+			(at 100.33 134.2969 0)
 			(show_name no)
 			(do_not_autoplace no)
@@
 		)
 		(property "Footprint" "Converter_ACDC:Converter_ACDC_Hahn_HS-400xx_THT"
-			(at 111.76 138.43 0)
+			(at 100.33 138.43 0)
 			(hide yes)
 			(show_name no)
@@
 		)
 		(property "Datasheet" ""
-			(at 111.76 138.43 0)
+			(at 100.33 138.43 0)
 			(hide yes)
 			(show_name no)
@@
 		)
 		(property "Description" "Power symbol creates a global label with name \"+5V\""
-			(at 111.76 138.43 0)
+			(at 100.33 138.43 0)
 			(hide yes)
 			(show_name no)
@@
 				)
 			)
+		)
+	)
+	(symbol
+		(lib_id "Diode:1N5817")
+		(at 107.95 140.97 180)
+		(unit 1)
+		(body_style 1)
+		(exclude_from_sim no)
+		(in_bom yes)
+		(on_board yes)
+		(in_pos_files yes)
+		(dnp no)
+		(fields_autoplaced yes)
+		(property "Reference" "D4"
+			(at 108.2675 135.5555 0)
+			(show_name no)
+			(do_not_autoplace no)
+			(effects
+				(font
+					(size 1.27 1.27)
+				)
+			)
+		)
+		(property "Value" "1N5817"
+			(at 108.2675 137.9798 0)
+			(show_name no)
+			(do_not_autoplace no)
+			(effects
+				(font
+					(size 1.27 1.27)
+				)
+			)
+		)
+		(property "Footprint" "Diode_THT:D_DO-41_SOD81_P10.16mm_Horizontal"
+			(at 107.95 136.525 0)
+			(hide yes)
+			(show_name no)
+			(do_not_autoplace no)
+			(effects
+				(font
+					(size 1.27 1.27)
+				)
+			)
+		)
+		(property "Datasheet" "http://www.vishay.com/docs/88525/1n5817.pdf"
+			(at 107.95 140.97 0)
+			(hide yes)
+			(show_name no)
+			(do_not_autoplace no)
+			(effects
+				(font
+					(size 1.27 1.27)
+				)
+			)
+		)
+		(property "Description" "20V 1A Schottky Barrier Rectifier Diode, DO-41"
+			(at 107.95 140.97 0)
+			(hide yes)
+			(show_name no)
+			(do_not_autoplace no)
+			(effects
+				(font
+					(size 1.27 1.27)
+				)
+			)
+		)
+		(pin "1"
+		)
+		(pin "2"
+		)
+		(instances
+			(project "Controller"
+				(path "/4060925a-c52c-48a2-a590-88d95c16dad5"
+					(reference "D4")
+					(unit 1)
+				)
+			)
